File: swadge-mx/swadge-mx-IMU.kicad_sch (KiCad schematic)
At the start: 5 parts, among them U5 LSM6DSL

Commit message: Updated power netclass, traces. Switched mic footprint. Added spk terminals
Other:
- note removed: "Inertial Measurement Unit (IMU)"
Changed lines of the file:
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@@
 	(generator_version "9.0")
 	(paper "A")
-	(rectangle
-		(start 83.82 38.1)
-		(end 119.38 43.18)
-		(stroke
-			(width 0)
-			(type solid)
-		)
-		(fill
-			(type color)
-			(color 191 255 127 1)
-		)
-	)
-	(text "Inertial Measurement Unit (IMU)"
-		(exclude_from_sim no)
-		(at 101.6 40.64 0)
-		(effects
-			(font
-				(size 1.27 1.27)
-			)
-		)
-	)
 	(text_box "LSM6DS3 I2C Addr = 0x6A"
 		(exclude_from_sim no)
